File: BB816-MATX-PCIE.kicad_sch (KiCad schematic)
At the start: 0 parts

Commit message: BankZero
Other:
- added sheet LCD Display (LCDDisplay.kicad_sch)
Changed lines of the file:
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@@
-(kicad_sch (version 20230121) (generator eeschema)
-  (paper "A4")
-  (sheet (at 185.42 115.57) (size 72.39 31.75) (fields_autoplaced)
-    (stroke (width 0.1524) (type solid))
-    (fill (color 0 0 0 0.0000))
-    (property "Sheetname" "BB816-MATX" (at 185.42 114.8584 0)
-      (effects (font (size 1.27 1.27)) (justify left bottom))
-    )
-    (property "Sheetfile" "BB816-MATX/BB816-MATX.kicad_sch" (at 185.42 147.9046 0)
-      (effects (font (size 1.27 1.27)) (justify left top))
-    )
-    (instances
-      (project "BB816-MATX-PCIE"
-        (path "/597c4a8d-3f77-42d9-910f-58b5c53fe80f" (page "2"))
-      )
-    )
-  )
-  (sheet (at 185.42 71.12) (size 73.66 30.48) (fields_autoplaced)
-    (stroke (width 0.1524) (type solid))
-    (fill (color 0 0 0 0.0000))
-    (property "Sheetname" "BB816-PCIE" (at 185.42 70.4084 0)
-      (effects (font (size 1.27 1.27)) (justify left bottom))
-    )
-    (property "Sheetfile" "BB816-PCIE/BB816-PCIE.kicad_sch" (at 185.42 102.1846 0)
-      (effects (font (size 1.27 1.27)) (justify left top))
-    )
-    (instances
-      (project "BB816-MATX-PCIE"
-        (path "/597c4a8d-3f77-42d9-910f-58b5c53fe80f" (page "3"))
-      )
-    )
-  )
-  (sheet_instances
-    (path "/" (page "1"))
-  )
+(kicad_sch
+	(version 20231120)
+	(generator "eeschema")
+	(generator_version "8.0")
+	(paper "A4")
+	(sheet
+		(at 185.42 115.57)
+		(size 72.39 31.75)
+		(fields_autoplaced yes)
+		(stroke
+			(width 0.1524)
+			(type solid)
+		)
+		(fill
+			(color 0 0 0 0.0000)
+		)
+		(property "Sheetname" "BB816-MATX"
+			(at 185.42 114.8584 0)
+			(effects
+				(font
+					(size 1.27 1.27)
+				)
+				(justify left bottom)
+			)
+		)
+		(property "Sheetfile" "BB816-MATX/BB816-MATX.kicad_sch"
+			(at 185.42 147.9046 0)
+			(effects
+				(font
+					(size 1.27 1.27)
+				)
+				(justify left top)
+			)
+		)
+		(instances
+			(project "BB816-MATX-PCIE"
+				(path "/597c4a8d-3f77-42d9-910f-58b5c53fe80f"
+					(page "2")
+				)
+			)
+		)
+	)
+	(sheet
+		(at 185.42 71.12)
+		(size 73.66 30.48)
+		(fields_autoplaced yes)
+		(stroke
+			(width 0.1524)
+			(type solid)
+		)
+		(fill
+			(color 0 0 0 0.0000)
+		)
+		(property "Sheetname" "BB816-PCIE"
+			(at 185.42 70.4084 0)
+			(effects
+				(font
+					(size 1.27 1.27)
+				)
+				(justify left bottom)
+			)
+		)
+		(property "Sheetfile" "BB816-PCIE/BB816-PCIE.kicad_sch"
+			(at 185.42 102.1846 0)
+			(effects
+				(font
+					(size 1.27 1.27)
+				)
+				(justify left top)
+			)
+		)
+		(instances
+			(project "BB816-MATX-PCIE"
+				(path "/597c4a8d-3f77-42d9-910f-58b5c53fe80f"
+					(page "3")
+				)
+			)
+		)
+	)
+	(sheet
+		(at 187.96 34.29)
+		(size 48.26 17.78)
+		(fields_autoplaced yes)
+		(stroke
+			(width 0.1524)
+			(type solid)
+		)
+		(fill
+			(color 0 0 0 0.0000)
+		)
+		(property "Sheetname" "LCD Display"
+			(at 187.96 33.5784 0)
+			(effects
+				(font
+					(size 1.27 1.27)
+				)
+				(justify left bottom)
+			)
+		)
+		(property "Sheetfile" "LCDDisplay.kicad_sch"
+			(at 187.96 52.6546 0)
+			(effects
+				(font
+					(size 1.27 1.27)
+				)
+				(justify left top)
+			)
+		)
+		(instances
+			(project "BB816-MATX-PCIE"
+				(path "/597c4a8d-3f77-42d9-910f-58b5c53fe80f"
+					(page "5")
+				)
+			)
+		)
+	)
+	(sheet_instances
+		(path "/"
+			(page "1")
+		)
+	)
 )
