File: BB816-MATX/BB816-MATX.kicad_pcb (KiCad board)
At the start: 4 copper layers, 243.8 x 243.8 mm, 17 parts, among them J1 10018783-10113TLF, J2 10018783-10113TLF, J3 10018783-10113TLF, J4 10018783-10113TLF, J5 39-28-1243, J6 Conn_02x40_Even_Odd, J7 PinSocket_1x02_P2.54mm_Vertic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, J8 PinSocket_2x18_P2.54mm_Vertic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

Commit message: doc
Parts:
- added J9: PWR_SW, Connector_PinSocket_2.54mm:PinSocket_1x02_P2.54mm_Vertical, F.Cu at (37.3, 220.3)
- J6: value Conn_02x40_Even_Odd -> PinSocket_2x40_P2.54mm_Vertical_Flip
Routing:
- net /PS_ON: track 0.00 -> 62.7 mm
Changed lines of the file:
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@@
+    )
+  )
+  (footprint "Connector_PinSocket_2.54mm:PinSocket_1x02_P2.54mm_Vertical" (layer "F.Cu")
+    (at 37.31 220.29)
+    (descr "Through hole straight socket strip, 1x02, 2.54mm pitch, single row (from Kicad 4.0.7), script generated")
+    (tags "Through hole socket strip THT 1x02 2.54mm single row")
+    (property "Sheetfile" "BB816-MATX.kicad_sch")
+    (property "Sheetname" "")
+    (property "ki_description" "Generic connector, single row, 01x02, script generated (kicad-library-utils/schlib/autogen/connector/)")
+    (property "ki_keywords" "connector")
+    (attr through_hole)
+    (fp_text reference "J9" (at 0 -2.77) (layer "F.SilkS")
+        (effects (font (size 1 1) (thickness 0.15)))
+    )
+    (fp_text value "PWR_SW" (at -2.36 1.26 270) (layer "F.Fab")
+        (effects (font (size 1 1) (thickness 0.15)))
+    )
+    (fp_text user "${REFERENCE}" (at 0 1.27 90) (layer "F.Fab")
+        (effects (font (size 1 1) (thickness 0.15)))
+    )
+    (fp_line (start -1.33 1.27) (end -1.33 3.87)
+      (stroke (width 0.12) (type solid)) (layer "F.SilkS"))
+    (fp_line (start -1.33 1.27) (end 1.33 1.27)
+      (stroke (width 0.12) (type solid)) (layer "F.SilkS"))
+    (fp_line (start -1.33 3.87) (end 1.33 3.87)
+      (stroke (width 0.12) (type solid)) (layer "F.SilkS"))
+    (fp_line (start 0 -1.33) (end 1.33 -1.33)
+      (stroke (width 0.12) (type solid)) (layer "F.SilkS"))
+    (fp_line (start 1.33 -1.33) (end 1.33 0)
+      (stroke (width 0.12) (type solid)) (layer "F.SilkS"))
+    (fp_line (start 1.33 1.27) (end 1.33 3.87)
+      (stroke (width 0.12) (type solid)) (layer "F.SilkS"))
+    (fp_line (start -1.8 -1.8) (end 1.75 -1.8)
+      (stroke (width 0.05) (type solid)) (layer "F.CrtYd"))
+    (fp_line (start -1.8 4.3) (end -1.8 -1.8)
+      (stroke (width 0.05) (type solid)) (layer "F.CrtYd"))
+    (fp_line (start 1.75 -1.8) (end 1.75 4.3)
+      (stroke (width 0.05) (type solid)) (layer "F.CrtYd"))
+    (fp_line (start 1.75 4.3) (end -1.8 4.3)
+      (stroke (width 0.05) (type solid)) (layer "F.CrtYd"))
+    (fp_line (start -1.27 -1.27) (end 0.635 -1.27)
+      (stroke (width 0.1) (type solid)) (layer "F.Fab"))
+    (fp_line (start -1.27 3.81) (end -1.27 -1.27)
+      (stroke (width 0.1) (type solid)) (layer "F.Fab"))
+    (fp_line (start 0.635 -1.27) (end 1.27 -0.635)
+      (stroke (width 0.1) (type solid)) (layer "F.Fab"))
+    (fp_line (start 1.27 -0.635) (end 1.27 3.81)
+      (stroke (width 0.1) (type solid)) (layer "F.Fab"))
+    (fp_line (start 1.27 3.81) (end -1.27 3.81)
+      (stroke (width 0.1) (type solid)) (layer "F.Fab"))
+    (pad "1" thru_hole rect (at 0 0) (size 1.7 1.7) (drill 1) (layers "*.Cu" "*.Mask")
+      (net 6 "/PS_ON") (pinfunction "Pin_1") (pintype "passive"))
+    (pad "2" thru_hole oval (at 0 2.54) (size 1.7 1.7) (drill 1) (layers "*.Cu" "*.Mask")
+      (net 1 "GND") (pinfunction "Pin_2") (pintype "passive"))
+    (model "${KICAD6_3DMODEL_DIR}/Connector_PinSocket_2.54mm.3dshapes/PinSocket_1x02_P2.54mm_Vertical.wrl"
+      (offset (xyz 0 0 0))
+      (scale (xyz 1 1 1))
+      (rotate (xyz 0 0 0))
     )
   )
@@
         (effects (font (size 1 1) (thickness 0.15)))
     )
-    (fp_text value "Conn_02x40_Even_Odd" (at 1.27 101.83) (layer "F.Fab") hide
+    (fp_text value "PinSocket_2x40_P2.54mm_Vertical_Flip" (at 1.27 101.83) (layer "F.Fab") hide
         (effects (font (size 1 1) (thickness 0.15)))
     )
@@
   (segment (start 88.6 216.1) (end 84.4 220.3) (width 0.146812) (layer "B.Cu") (net 5))
   (segment (start 84.4 220.3) (end 84.4 221.6) (width 0.146812) (layer "B.Cu") (net 5))
+  (segment (start 37.31 220.29) (end 38.73 220.29) (width 0.146812) (layer "F.Cu") (net 6))
+  (segment (start 94.21 224.52) (end 97.05 221.68) (width 0.146812) (layer "F.Cu") (net 6))
+  (segment (start 38.73 220.29) (end 42.96 224.52) (width 0.146812) (layer "F.Cu") (net 6))
+  (segment (start 42.96 224.52) (end 94.21 224.52) (width 0.146812) (layer "F.Cu") (net 6))
   (segment (start 53.2792 69.39) (end 52.23 70.4392) (width 0.146812) (layer "F.Cu") (net 10))
   (segment (start 113.2248 70.4792) (end 112.1756 69.43) (width 0.146812) (layer "F.Cu") (net 10))
@@
     (connect_pads (clearance 0.508))
     (min_thickness 0.25) (filled_areas_thickness no)
-    (fill (thermal_gap 0.5) (thermal_bridge_width 0.5))
+    (fill yes (thermal_gap 0.5) (thermal_bridge_width 0.5))
     (polygon
       (pts
@@
     (connect_pads (clearance 0.508))
     (min_thickness 0.25) (filled_areas_thickness no)
-    (fill (thermal_gap 0.5) (thermal_bridge_width 0.5))
+    (fill yes (thermal_gap 0.5) (thermal_bridge_width 0.5))
     (polygon
       (pts

Commit message: BankZero
Parts:
- added C1: 220u, Capacitor_THT:CP_Radial_D6.3mm_P2.50mm, F.Cu at (104.1, 213.2)
- added C2: 220u, Capacitor_THT:CP_Radial_D6.3mm_P2.50mm, F.Cu at (72.5, 61.0)
- added C3: 220u, Capacitor_THT:CP_Radial_D6.3mm_P2.50mm, F.Cu at (134.7, 61.3)
- added C4: 220u, Capacitor_THT:CP_Radial_D6.3mm_P2.50mm, F.Cu at (92.7, 60.8)
- added C5: 220u, Capacitor_THT:CP_Radial_D6.3mm_P2.50mm, F.Cu at (113.2, 60.8)
- added C6: 220u, Capacitor_THT:CP_Radial_D6.3mm_P2.50mm, F.Cu at (52.5, 61.0)
- added C7: 220u, Capacitor_THT:CP_Radial_D6.3mm_P2.50mm, F.Cu at (157.6, 60.1)
- added J10: BB816_Breakout_A27, BB816-MATX-PCIE:BB816_Breakout_A27_Socket_NO_VDPA, F.Cu at (154.8, 68.3)
- added J11: PinSocket_1x02_P2.54mm_Vertical, Connector_PinSocket_2.54mm:PinSocket_1x02_P2.54mm_Vertical, F.Cu at (111.7, 213.1)
- moved J5 27.5 mm to (95.1, 215.2), turned to 180 degrees
- moved J7 21.7 mm to (114.2, 213.1)
- moved J9 7.38 mm to (38.2, 213.0)
Routing:
- net /PS_ON: track 62.7 -> 0.00 mm
- net /+3.3v: track 29.6 -> 0.00 mm
- net /A5: track 139.9 -> 163.9 mm
- net /A13: track 125.3 -> 149.2 mm
- net /~{RST}: track 87.5 -> 111.4 mm
- net /D6: track 155.6 -> 179.5 mm
- net /D4: track 158.8 -> 182.7 mm
- net /D2: track 162.0 -> 185.9 mm
- net /A4: track 146.6 -> 170.5 mm
- net /A20: track 119.1 -> 143.0 mm
- net /A10: track 134.7 -> 158.6 mm
- net /A0: track 152.6 -> 176.5 mm
- net /~{VP}: track 106.7 -> 130.6 mm
- net /~{RD}: track 97.5 -> 121.4 mm
- net /~{ML}: track 113.0 -> 136.9 mm
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