File: BB816-PCIE-BANKZERO/BB816-PCIE-BANKZERO.kicad_sch (KiCad schematic)
At the start: 22 parts, among them J1 SPI_0, J2 LCD Display, J3 LCD Backlight, J4 SPI_1, J5 GPIO, U1 AS7C256B-15PIN, U2 AS7C256B-15PIN, U3 AT28C256-15PU, U4 74HC138, U5 74HC138, U6 74HC148, U7 74HC244, U8 74HC283, U9 W65C22SxP

Commit message: big commit
Parts:
- removed D2, D3: 1N5817, Diode_THT:D_DO-41_SOD81_P10.16mm_Horizontal, symbol Diode:1N5817
- removed J1: SPI_0, Connector_PinHeader_2.54mm:PinHeader_1x06_P2.54mm_Horizontal, symbol BB816-MATX-PCIE:SPI_Header
- removed J2: LCD Display, Connector_PinSocket_2.54mm:PinSocket_1x16_P2.54mm_Horizontal, symbol BB816-MATX-PCIE:LCD_Display_Header
- removed J3: LCD Backlight, Connector_PinHeader_2.54mm:PinHeader_1x03_P2.54mm_Horizontal, symbol BB816-MATX-PCIE:LCD_Backlight_Header
- removed J4: SPI_1, Connector_PinHeader_2.54mm:PinHeader_1x06_P2.54mm_Horizontal, symbol BB816-MATX-PCIE:SPI_Header
- removed J5: GPIO, Connector_PinHeader_2.54mm:PinHeader_1x05_P2.54mm_Horizontal, symbol Connector_Generic:Conn_01x05
- removed R1: 3.3K, symbol Device:R
- removed U5: 74HC138, Package_DIP:DIP-16_W7.62mm_Socket, symbol BB816-MATX-PCIE:74HC138
- removed U6: 74HC148, Package_DIP:DIP-16_W7.62mm_Socket, symbol BB816-MATX-PCIE:74HC148
- removed U7: 74HC244, Package_DIP:DIP-20_W7.62mm_Socket, symbol BB816-MATX-PCIE:74HC244
- removed U8: 74HC283, Package_DIP:DIP-16_W7.62mm_Socket, symbol BB816-MATX-PCIE:74HC283
- removed U9: W65C22SxP, Package_DIP:DIP-40_W15.24mm_Socket, symbol BB816:W65C22SxP
- added J1: Bypass, Connector_PinHeader_2.54mm:PinHeader_2x04_P2.54mm_Vertical, symbol Connector_Generic:Conn_02x04_Odd_Even
- added U10, U16: 74HC138, Package_DIP:DIP-16_W7.62mm_Socket, symbol BB816-MATX-PCIE:74HC138
- added U15, U9: 74HC32, Package_DIP:DIP-14_W7.62mm_Socket, symbol BB816-MATX-PCIE:74HC32
- added U18: 74HC00, symbol BB816-MATX-PCIE:74HC08
- added U23: 74HC04, Package_DIP:DIP-14_W7.62mm_Socket, symbol 74xx:74HC04
- added U5: 74HC148, Package_DIP:DIP-16_W7.62mm_Socket, symbol BB816-MATX-PCIE:74HC148
- added U6: 74HC125, Package_DIP:DIP-14_W7.62mm_Socket, symbol BB816-MATX-PCIE:74HC125
- added U7: 74HC283, Package_DIP:DIP-16_W7.62mm_Socket, symbol BB816-MATX-PCIE:74HC283
- R2, R3, R4: footprint (none) -> Resistor_THT:R_Axial_DIN0207_L6.3mm_D2.5mm_P7.62mm_Horizontal
- U1, U2: footprint PDIP-28_MIL300_ALL -> Package_DIP:DIP-28_W7.62mm_Socket
Connections:
- net ~{RAM1_OE} is gone; now on net ~{RAM0_OE}: U2.22 (*OE)
- net ~{RAM1_WE} is gone; now on net ~{RAM0_WE}: U2.27 (*WE)
- net ~{ROM_OE} is gone; now on net ~{RAM0_OE}: U3.22 (~OE)
- net ~{ROM_WE} is gone; now on net ~{RAM0_WE}: U3.27 (~WE)
- net A1: now also U4.6 (G1), J1.7 (Pin_7), U7.5 (A1); no longer U4.1 (A)
- net A10: now also U10.1 (A)
- net A11: now also U10.2 (B)
- net A12: now also U10.3 (C)
- net A13: now also U10.6 (G1)
- net A14: now also U23.11
- net A2: now also U4.1 (A), J1.5 (Pin_5), U7.3 (A2); no longer U4.2 (B)
- net A3: now also U4.2 (B), J1.3 (Pin_3), U7.14 (A3); no longer U4.3 (C)
- net A4: now also U4.3 (C), J1.1 (Pin_1), U7.12 (A4)
- net A5: now also U16.1 (A)
- net A6: now also U16.2 (B)
- net A7: now also U16.3 (C)
- net A8: now also U9.10
- net A9: now also U23.9
- net AA1: now also J1.8 (Pin_8), U7.4 (S1)
- net AA2: now also J1.6 (Pin_6), U7.1 (S2)
- net AA3: now also J1.4 (Pin_4), U7.13 (S3)
- net AA4: now also J1.2 (Pin_2), U7.10 (S4)
- net D0: now also U3.11 (I/O0); no longer U3.19 (I/O7)
- net D1: now also U3.12 (I/O1); no longer U3.18 (I/O6)
- net D2: now also U3.13 (I/O2); no longer U3.17 (I/O5)
- net D3: now also U3.15 (I/O3); no longer U3.16 (I/O4)
- net D4: now also U3.16 (I/O4); no longer U3.15 (I/O3)
- net D5: now also U3.17 (I/O5); no longer U3.13 (I/O2)
- net D6: now also U3.18 (I/O6); no longer U3.12 (I/O1)
- net D7: now also U3.19 (I/O7); no longer U3.11 (I/O0)
- net E: now also U4.4 (~{G}2A), U18.2, U23.5; no longer U4.6 (G1)
- net GND: now also U10.8 (GND), U15.12, U15.13, U15.7 (GND), U16.8 (GND), U18.10, U18.7 (GND), U18.9, U23.7 (GND), U5.8 (GND), U6.7 (GND), U6.9, U7.11 (B4), U7.7 (C0), U7.8 (GND), U9.7 (GND)
- net VCC: now also RN1.1 (common), U10.16 (VCC), U15.14 (VCC), U16.16 (VCC), U16.6 (G1), U18.14 (VCC), U23.14 (VCC), U5.16 (VCC), U6.10, U6.14 (VCC), U7.16 (VCC), U9.14 (VCC)
- net ~{IRQ0}: now also U5.4 (I7)
- net ~{IRQ1}: now also U5.3 (I6)
- net ~{IRQ2}: now also U5.2 (I5)
- net ~{IRQ3}: now also U5.1 (I4)
- net ~{IRQ4}: now also U5.13 (I3)
- net ~{IRQ5}: now also U5.12 (I2)
- net ~{IRQ6}: now also U5.11 (I1)
- net ~{IRQ7}: now also U5.10 (IO)
- net ~{IRQ}: now also D1.2 (A)
- net ~{RAM0_CE}: now also U9.3
- net ~{RAM0_OE}: now also U23.1
- net ~{RAM1_CE}: now also U15.6
- net ~{ROM_CE}: now also U15.8
- net ~{VP}: no longer U4.4 (~{G}2A)
- net ~{VP_IRQ}: now reaches U4.12 (Y3)
- net ~{VP_IRQ}: now also U5.5 (EI)
- net at D1.1 (K): now also U5.14 (GS), U6.1, U6.13, U6.4
- net OFF3: now reaches R4.1
- net OFF3: now also U6.11, U7.15 (B3)
- net OFF2: now reaches R3.1
- net OFF2: now also U6.3, U7.2 (B2)
- net OFF1: now reaches R2.1
- net OFF1: now also U6.6, U7.6 (B1)
- new net: U5.6 (S2), U6.12
- new net: U5.7 (S1), U6.2
- new net: U5.9 (S0), U6.5
- new net: U9.5, U9.8
- new net: U10.7 (Y7), U9.4
- new net: U18.12, U18.13, U18.4, U18.5
- new net A15: U23.13, U9.2
- new net EMU_RD: U15.4, U18.3
- new net IO_PAGE: U15.1, U23.4
- new net RD: U18.1, U23.2
- new net ~{32K_HI_MEM}: U15.3, U15.5, U15.9
- new net ~{32K_HI}: U10.4 (~{G}2A), U15.2, U9.11
- new net ~{A14}: U10.5 (~{G}2B), U23.10
- new net ~{A15}: U23.12, U9.13
- new net ~{A9}: U23.8, U9.9
- new net ~{BANK0}: U9.1, U9.12
- new net ~{E}: U15.10, U23.6
- new net ~{IOCS0}: U16.15 (Y0)
- new net ~{IOCS1}: U16.14 (Y1)
- new net ~{IOCS2}: U16.13 (Y2)
- new net ~{IOCS3}: U16.12 (Y3)
- new net ~{IOCS4}: U16.11 (Y4)
- new net ~{IOCS5}: U16.10 (Y5)
- new net ~{IOCS6}: U16.9 (Y6)
- new net ~{IOCS7}: U16.7 (Y7)
- new net ~{IO_PAGE}: U16.4 (~{G}2A), U16.5 (~{G}2B), U23.3, U9.6
- no-connect marks 10 -> 21
Other:
- note added: "$0000-$7FFF 32K RAM0 $8000-$FFFF 32K RAM1 Emulation: Write-Only Native: Read-Write) $8000-$FFFF 32K ROM Emulation: Read-Write Native: Disabled) $FE00-$FEFF I/O Area (8x32 byte devices)"
- note added: "$E or $F"
- note added: "$E*"
- note added: "$FE00 ~{IOCS0} $FE20 ~{IOCS1} $FE40 ~{IOCS2} $FE60 ~{IOCS3} $FE80 ~{IOCS4} $FEA0 ~{IOCS5} $FEC0 ~{IOCS6} $FEE0 ~{IOCS7}"
- note added: "*or $C, can't happen during ~{VP}"
- note added: "A15 High"
- note added: "A15 Low"
- note added: "A3-A1 Offset"
- note added: "Address Decode"
- note added: "After $FFE4 COP $FFE6 BRK $FFE8 ABORT $FFEA NMI $FFEE IRQ0 $FFF0 IRQ1 $FFF2 IRQ2 $FFF4 IRQ3 $FFF6 IRQ4 $FFF8 IRQ5 $FFFA IRQ6 $FFFC RESET"
- note added: "Assumes EEPROM write protect"
- note added: "BANK0 LO/HI 32K Detect"
- note added: "Bank Zero"
- note added: "Bank Zero RAM + ROM"
- note added: "Before $FFE4 COP $FFE6 BRK $FFE8 ABORT $FFEA NMI $FFEE IRQ $FFFC RESET"
- note added: "Buffered A3-A1 Offset"
- note added: "E low (65816 native mode) VP low (Vector Pull is taking place) A1 high (pulling LSB of vector)"
- note added: "Emulation Mode (E High)"
- note added: "I/O Map"
- note added: "I/O Page $FE Detect"
- note added: "IRQ Vector Offset [0-7]x2"
- note added: "IRQ Vector Pull Rewrite"
- note added: "Native Mode (E Low)"
- note added: "RAM/ROM Control"
- note added: "RAM0"
- note added: "RAM0 Enabled"
- note added: "RAM1"
- note added: "ROM"
- note added: "R~{W} high (read)"
- note added: "R~{W} low (write)"
- note added: "Suppress ROM ~{CE} in Native mode"
- note added: "Suppress read from RAM1 in Emulation mode"
- note added: "~{BANK0} and ~{CS0} Low (Board Enabled)"
- note added: "~{RAM0_CE} high"
- note added: "~{RAM0_CE} low ~{RAM0_WE} = R/~{W} ~{RAM0_OE} = ~{R}/W"
- note added: "~{RAM1_CE} high"
- note added: "~{RAM1_CE} high ~{RAM1_WE} high ~{RAM1_OE} high"
- note added: "~{RAM1_CE} low ~{RAM1_WE} high ~{RAM1_OE} low"
- note added: "~{RAM1_CE} low ~{RAM1_WE} low ~{RAM1_OE} high"
- note added: "~{ROM_CE} high"
- note added: "~{ROM_CE} high ~{ROM_WE} high ~{ROM_OE} high"
- note added: "~{ROM_CE} low ~{ROM_WE} high ~{ROM_OE} low"
- note added: "~{ROM_CE} low ~{ROM_WE} low ~{ROM_OE} high"
- note added: "~{STRETCH_RQ} high"
- note added: "~{STRETCH_RQ} low"
- note added: "~{VP} E A7 A6 A5 A4 A3 A2 A1 A0 L L H H X L H H H X"
- note removed: "Bank Zero RAM/ROM"
- note removed: "Console I/O + SPI"
- note removed: "Emulation $FFE0 BRK/IRQ1 $FFE2 BRK/IRQ2 $FFE4 BRK/IRQ3 $FFE6 BRK/IRQ4 $FFE8 BRK/IRQ5 $FFEA BRK/IRQ6 $FFEC BRK/IRQ7 ... $FFF4 NMI $FFFC RESET $FFFE IRQ0"
- note removed: "Emulation $FFF4 NMI $FFFC RESET $FFFE IRQ0"
- note removed: "Native $FFE4 COP $FFE6 BRK $FFE8 ABORT $FFEA NMI $FFEE IRQ $FFFC RESET"
- note removed: "Native $FFE4 COP $FFE6 BRK $FFE8 ABORT $FFEA NMI $FFEE IRQ0 $FFF0 IRQ1 $FFF2 IRQ2 $FFF4 IRQ3 $FFF6 IRQ4 $FFF8 IRQ5 $FFFA IRQ6 $FFFC RESET"
- note removed: "Rewritten Vector Address"
- note removed: "Vector Addresses (Datasheet)"
- note removed: "Vector Pull Rewrite"
- moved on the sheet: U1, U2, U3

Commit message: Bum AND
Parts:
- removed U18: 74HC00, symbol BB816-MATX-PCIE:74HC08
- removed unit 1 of U23
Connections:
- net E: now also U6.9
- net EMU_RD: now also U6.8
- net GND: no longer U6.9
- net VCC: no longer U6.10
- net ~{RAM0_OE}: now also U6.10
- no-connect marks 21 -> 19
Other:
- note added: "E low (65816 native mode) VP low (Vector Pull active) A1 high"
- note removed: "E low (65816 native mode) VP low (Vector Pull is taking place) A1 high (pulling LSB of vector)"

Commit message: Cleanup
Parts:
- added R1: 3.3K, Resistor_THT:R_Axial_DIN0207_L6.3mm_D2.5mm_P7.62mm_Horizontal, symbol Device:R
Connections:
- net EMU_RD: now also R1.1
- net GND: now also R1.2
Other:
- note added: "~{VP} E A7 A6 A5 A4 A3 A2 A1 A0 L L H H H L H H H X"
- note removed: "~{VP} E A7 A6 A5 A4 A3 A2 A1 A0 L L H H X L H H H X"
- moved on the sheet: D1, J1, R2, R3, R4, RN1, U1, U15D, U15E, U2, U23G, U3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

Commit message: Bad PCB
Parts:
- added U11, U12: W65C51NxP, symbol BB816-MATX-PCIE:W65C51NxP
- added U8: W65C22SxP, symbol BB816-MATX-PCIE:W65C22SxP
Other:
- moved on the sheet: R1, U10, U15A, U15B, U15C, U15D, U15E, U16, U23B, U23C, U23D, U23E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

Commit message: Add VIA and ACIA
Parts:
- U11, U12: footprint (none) -> Package_DIP:DIP-28_W15.24mm_Socket
- U8: footprint (none) -> Package_DIP:DIP-40_W15.24mm_Socket
Connections:
- no-connect marks 19 -> 18
Changed lines of the file:
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@@
 		(at 72.39 248.92)
 	)
-	(no_connect
-		(at 64.77 214.63)
-	)
 	(bus_entry
 		(at 208.28 147.32)
@@
 		)
 	)
-	(wire
-		(pts
-			(xy 43.18 218.44) (xy 43.18 220.98)
-		)
-		(stroke
-			(width 0)
-			(type default)
-		)
-	)
 	(bus
 		(pts
@@
 	(wire
 		(pts
-			(xy 57.15 220.98) (xy 43.18 220.98)
-		)
-		(stroke
-			(width 0)
-			(type default)
-		)
-	)
-	(wire
-		(pts
 			(xy 207.01 213.36) (xy 201.93 213.36)
 		)
@@
 	)
 	(symbol
-		(lib_id "power:GND")
-		(at 49.53 214.63 0)
-		(unit 1)
-		(exclude_from_sim no)
-		(in_bom yes)
-		(on_board yes)
-		(dnp no)
-		(property "Reference" "#PWR027"
-			(at 49.53 220.98 0)
-			(effects
-				(font
-					(size 1.27 1.27)
-				)
-				(hide yes)
-			)
-		)
-		(property "Value" "GND"
-			(at 49.657 219.0242 0)
-			(effects
-				(font
-					(size 1.27 1.27)
-				)
-			)
-		)
-		(property "Footprint" ""
-			(at 49.53 214.63 0)
-			(effects
-				(font
-					(size 1.27 1.27)
-				)
-				(hide yes)
-			)
-		)
-		(property "Datasheet" ""
-			(at 49.53 214.63 0)
-			(effects
-				(font
-					(size 1.27 1.27)
-				)
-				(hide yes)
-			)
-		)
-		(property "Description" ""
-			(at 49.53 214.63 0)
-			(effects
-				(font
-					(size 1.27 1.27)
-				)
-				(hide yes)
-			)
-		)
-		(pin "1"
-		)
-		(instances
-			(project "BB816-PCIE-BANKZERO"
-				(path "/7d7ddd8d-6afe-4f94-a79c-e7b1fbf309ce"
-					(reference "#PWR027")
-					(unit 1)
-				)
-			)
-		)
-	)
-	(symbol
 		(lib_id "power:VCC")
 		(at 217.17 198.12 270)
@@
 			)
 		)
-		(property "Footprint" ""
+		(property "Footprint" "Package_DIP:DIP-28_W15.24mm_Socket"
 			(at 351.79 143.51 0)
 			(effects
@@
 			)
 		)
-		(property "Footprint" ""
+		(property "Footprint" "Package_DIP:DIP-40_W15.24mm_Socket"
 			(at 320.04 66.04 0)
 			(effects
@@
 			)
 		)
-		(property "Footprint" ""
+		(property "Footprint" "Package_DIP:DIP-28_W15.24mm_Socket"
 			(at 303.53 142.24 0)
 			(effects
@@
 				)
 			)
-		)
-	)
-	(symbol
-		(lib_id "power:VCC")
-		(at 43.18 218.44 0)
-		(unit 1)
-		(exclude_from_sim no)
-		(in_bom yes)
-		(on_board yes)
-		(dnp no)
-		(fields_autoplaced yes)
-		(property "Reference" "#PWR014"
-			(at 43.18 222.25 0)
-			(effects
-				(font
-					(size 1.27 1.27)
-				)
-				(hide yes)
-			)
-		)
-		(property "Value" "VCC"
-			(at 43.18 213.36 0)
-			(effects
-				(font
-					(size 1.27 1.27)
-				)
-			)
-		)
-		(property "Footprint" ""
-			(at 43.18 218.44 0)
-			(effects
-				(font
-					(size 1.27 1.27)
-				)
-				(hide yes)
-			)
-		)
-		(property "Datasheet" ""
-			(at 43.18 218.44 0)
-			(effects
-				(font
-					(size 1.27 1.27)
-				)
-				(hide yes)
-			)
-		)
-		(property "Description" "Power symbol creates a global label with name \"VCC\""
-			(at 43.18 218.44 0)
-			(effects
-				(font
-					(size 1.27 1.27)
-				)
-				(hide yes)
-			)
-		)
-		(pin "1"
-		)
-		(instances
-			(project "BB816-PCIE-BANKZERO"
-				(path "/7d7ddd8d-6afe-4f94-a79c-e7b1fbf309ce"
-					(reference "#PWR014")
-					(unit 1)
-				)
-			)

Commit message: VIA
Parts:
- removed U11: W65C51NxP, Package_DIP:DIP-28_W15.24mm_Socket, symbol BB816-MATX-PCIE:W65C51NxP
- added J2: Conn_01x22_Pin, Connector_PinHeader_2.54mm:PinHeader_1x22_P2.54mm_Horizontal, symbol Connector:Conn_01x22_Pin
Connections:
- net A0: now also U8.38 (RS0)
- net A1: now also U8.37 (RS1)
- net A2: now also U8.36 (RS2)
- net A3: now also U8.35 (RS3)
- net D0: now also U8.33 (D0)
- net D1: now also U8.32 (D1)
- net D2: now also U8.31 (D2)
- net D3: now also U8.30 (D3)
- net D4: now also U8.29 (D4)
- net D5: now also U8.28 (D5)
- net D6: now also U8.27 (D6)
- net D7: now also U8.26 (D7)
- net GND: now also U8.1 (VSS)
- net VCC: now also U8.20 (VCC), U8.24 (CS1)
- net ~{IOCS0}: now also U8.23 (~{CS2})
- net ~{IRQ0}: now also U8.21 (~{IRQ})
- net ~{RAM0_WE}: now also U8.22 (R/~{W})
- net at U8.10 (PB0): now also J2.13 (Pin_13)
- net at U8.11 (PB1): now also J2.14 (Pin_14)
- net at U8.12 (PB2): now also J2.15 (Pin_15)
- net at U8.13 (PB3): now also J2.16 (Pin_16)
- net at U8.14 (PB4): now also J2.17 (Pin_17)
- net at U8.15 (PB5): now also J2.18 (Pin_18)
- net at U8.16 (PB6): now also J2.19 (Pin_19)
- net at U8.17 (PB7): now also J2.20 (Pin_20)
- net at U8.18 (CB1): now also J2.21 (Pin_21)
- net at U8.19 (CB2): now also J2.22 (Pin_22)
- net at U8.2 (PA0): now also J2.3 (Pin_3)
- net at U8.3 (PA1): now also J2.4 (Pin_4)
- net at U8.39 (CA2): now also J2.12 (Pin_12)
- net at U8.4 (PA2): now also J2.5 (Pin_5)
- net at U8.40 (CA1): now also J2.11 (Pin_11)
- net at U8.5 (PA3): now also J2.6 (Pin_6)
- net at U8.6 (PA4): now also J2.7 (Pin_7)
- net at U8.7 (PA5): now also J2.8 (Pin_8)
- net at U8.8 (PA6): now also J2.9 (Pin_9)
- net at U8.9 (PA7): now also J2.10 (Pin_10)
Other:
- note added: "VIA"
- moved on the sheet: U12

Commit message: Stuff
Parts:
- J2: footprint Connector_PinHeader_2.54mm:PinHeader_1x22_P2.54mm_Horizontal -> Connector_PinSocket_2.54mm:PinSocket_1x22_P2.54mm_Horizontal
Connections:
- net GND: now also J2.2 (Pin_2)
- net VCC: now also J2.1 (Pin_1)
- net PB0: now reaches J2.13 (Pin_13), U8.10 (PB0)
- net PB1: now reaches J2.14 (Pin_14), U8.11 (PB1)
- net PB2: now reaches J2.15 (Pin_15), U8.12 (PB2)
- net PB3: now reaches J2.16 (Pin_16), U8.13 (PB3)
- net PB4: now reaches J2.17 (Pin_17), U8.14 (PB4)
- net PB5: now reaches J2.18 (Pin_18), U8.15 (PB5)
- net PB6: now reaches J2.19 (Pin_19), U8.16 (PB6)
- net PB7: now reaches J2.20 (Pin_20), U8.17 (PB7)
- net CB1: now reaches J2.21 (Pin_21), U8.18 (CB1)
- net CB2: now reaches J2.22 (Pin_22), U8.19 (CB2)
- net CA1: now reaches J2.3 (Pin_3)
- net CA1: now also U8.40 (CA1); no longer U8.2 (PA0)
- net CLK: now reaches U8.25 (ϕ2)
- net CA2: now reaches J2.4 (Pin_4)
- net CA2: now also U8.39 (CA2); no longer U8.3 (PA1)
- net PA7: now reaches J2.12 (Pin_12)
- net PA7: now also U8.9 (PA7); no longer U8.39 (CA2)
- net PA0: now reaches J2.5 (Pin_5)
- net PA0: now also U8.2 (PA0); no longer U8.4 (PA2)
- net PA6: now reaches J2.11 (Pin_11)
- net PA6: now also U8.8 (PA6); no longer U8.40 (CA1)
- net PA1: now reaches J2.6 (Pin_6)
- net PA1: now also U8.3 (PA1); no longer U8.5 (PA3)
- net PA2: now reaches J2.7 (Pin_7)
- net PA2: now also U8.4 (PA2); no longer U8.6 (PA4)
- net PA3: now reaches J2.8 (Pin_8)
- net PA3: now also U8.5 (PA3); no longer U8.7 (PA5)
- net PA4: now reaches J2.9 (Pin_9)
- net PA4: now also U8.6 (PA4); no longer U8.8 (PA6)
- net PA5: now reaches J2.10 (Pin_10)
- net PA5: now also U8.7 (PA5); no longer U8.9 (PA7)
Other:
- note added: "ACIA"
- note removed: "A15 High"
- note removed: "A15 Low"
- note removed: "Assumes EEPROM write protect"
- note removed: "Emulation Mode (E High)"
- note removed: "Native Mode (E Low)"
- note removed: "RAM0 Enabled"
- note removed: "R~{W} high (read)"
- note removed: "R~{W} low (write)"
- note removed: "~{BANK0} and ~{CS0} Low (Board Enabled)"
- note removed: "~{RAM0_CE} high"
- note removed: "~{RAM0_CE} low ~{RAM0_WE} = R/~{W} ~{RAM0_OE} = ~{R}/W"
- note removed: "~{RAM1_CE} high"
- note removed: "~{RAM1_CE} high ~{RAM1_WE} high ~{RAM1_OE} high"
- note removed: "~{RAM1_CE} low ~{RAM1_WE} high ~{RAM1_OE} low"
- note removed: "~{RAM1_CE} low ~{RAM1_WE} low ~{RAM1_OE} high"
- note removed: "~{ROM_CE} high"
- note removed: "~{ROM_CE} high ~{ROM_WE} high ~{ROM_OE} high"
- note removed: "~{ROM_CE} low ~{ROM_WE} high ~{ROM_OE} low"
- note removed: "~{ROM_CE} low ~{ROM_WE} low ~{ROM_OE} high"
- note removed: "~{STRETCH_RQ} high"
- note removed: "~{STRETCH_RQ} low"
- moved on the sheet: J2, U12
